Commit message: cylinder primitive added

File: src/teleop_arm/urdf/cylinder.urdf (robot description, URDF)
Before this commit: robot small_cylinder, 1 links, 0 joints
Links:
- added link wedge_link, mass 0.02; collision cylinder length=0.02 radius=0.03; visual cylinder length=0.02 radius=0.035
- link cylinder_link: geometry collision cylinder length=0.5 radius=0.025; visual cylinder length=0.5 radius=0.025
Joints:
- added joint wedge_joint: type fixed, parent cylinder_link, child wedge_link, origin xyz=0 0 0.2 rpy=0 0 0
