Commit message: fixed structure

File: Arm_Urdf/old_arm_description/urdf/urdf/arm_urdf.urdf (robot description, URDF)
Before this commit: robot arm_urdf, 7 links, 6 joints
Links:
- link base_link: geometry collision mesh filename=package://Arm_Urdf/old_arm_description/meshes/base_link.STL; visual mesh filename=package://Arm_Urdf/old_arm_description/meshes/base_link.STL
- link link_0: geometry collision mesh filename=package://Arm_Urdf/old_arm_description/meshes/link_0.STL; visual mesh filename=package://Arm_Urdf/old_arm_description/meshes/link_0.STL
- link link_1: geometry collision mesh filename=package://Arm_Urdf/old_arm_description/meshes/link_1.STL; visual mesh filename=package://Arm_Urdf/old_arm_description/meshes/link_1.STL
- link link_2: geometry collision mesh filename=package://Arm_Urdf/old_arm_description/meshes/link_2.STL; visual mesh filename=package://Arm_Urdf/old_arm_description/meshes/link_2.STL
- link link_3: geometry collision mesh filename=package://Arm_Urdf/old_arm_description/meshes/link_3.STL; visual mesh filename=package://Arm_Urdf/old_arm_description/meshes/link_3.STL
- link link_4: geometry collision mesh filename=package://Arm_Urdf/old_arm_description/meshes/link_4.STL; visual mesh filename=package://Arm_Urdf/old_arm_description/meshes/link_4.STL
