Commit message: stereo vision added

File: Arm_Urdf/urdf/Arm_Urdf.urdf (robot description, URDF)
Before this commit: robot Arm_Urdf, 12 links, 11 joints
Joints:
- joint camera_joint1: origin xyz=0.0 -0.02 0.02 rpy=0 0 -1.57 -> xyz=-0.03 -0.082 0.012 rpy=0 -1.57 1.57; parent Link_1 -> Link_6
- joint camera_joint2: origin xyz=0.0 -0.082 0.012 rpy=0 -1.57 1.57 -> xyz=0.03 -0.082 0.012 rpy=0 -1.57 1.57

Commit message: servoing fixed

File: Arm_Urdf/urdf/Arm_Urdf.urdf (robot description, URDF)
Before this commit: robot Arm_Urdf, 12 links, 11 joints
Links:
- added link camera_optical_link
Joints:
- added joint camera_optical_joint: type fixed, parent camera_link1, child camera_optical_link, origin xyz=0.0 0.0 0.0 rpy=0 -3.14132 -1.57

Commit message: Fixed frame

File: Arm_Urdf/urdf/Arm_Urdf.urdf (robot description, URDF)
Before this commit: robot Arm_Urdf, 13 links, 12 joints
Links:
- removed link camera_optical_link
Joints:
- removed joint camera_optical_joint

Commit message: improved visual servoing

File: Arm_Urdf/urdf/Arm_Urdf.urdf (robot description, URDF)
Before this commit: robot Arm_Urdf, 12 links, 11 joints
Links:
- added link camera_optical_link1
- added link camera_optical_link2
Joints:
- added joint camera_optical_joint1: type fixed, parent camera_link1, child camera_optical_link1, origin xyz=0 0 0 rpy=1.57 0 1.57, axis 0 1 0
- added joint camera_optical_joint2: type fixed, parent camera_link2, child camera_optical_link2, origin xyz=0 0 0 rpy=1.57 0 1.57, axis 0 1 0
