Commit message: depth camera urdf added

File: src/Arm_Urdf/urdf/Arm_Urdf.urdf (robot description, URDF)
Before this commit: robot Arm_Urdf, 18 links, 17 joints
Links:
- added link realsense_camera_link; visual box size=0.08 0.03 0.02
Joints:
- added joint realsense_fixed_joint: type fixed, parent left_camera_link, child realsense_camera_link, origin xyz=0.1 0 0 rpy=0 0 0

Commit message: depth camera function added (it is giving wrong coordinates)

File: src/Arm_Urdf/urdf/Arm_Urdf.urdf (robot description, URDF)
Before this commit: robot Arm_Urdf, 19 links, 18 joints
Links:
- link realsense_camera_link: mass None -> 1e-5; geometry collision box size=0.025 0.025 0.025; visual box size=0.025 0.025 0.025
Joints:
- joint realsense_fixed_joint: axis (none) -> 0 1 0; origin xyz=0.1 0 0 rpy=0 0 0 -> xyz=0 -0.095 0.012 rpy=0 -1.57 1.57; parent left_camera_link -> Link_6

Commit message: updated autonomous package from autonomous pipeline

File: src/Arm_Urdf/urdf/Arm_Urdf.urdf (robot description, URDF)
Before this commit: robot Arm_Urdf, 19 links, 18 joints
Links:
- removed link realsense_camera_link
Joints:
- removed joint realsense_fixed_joint

Commit message: arm is able to type now

File: src/Arm_Urdf/urdf/Arm_Urdf.urdf (robot description, URDF)
Before this commit: robot Arm_Urdf, 18 links, 17 joints
Links:
- removed link Gripper_1
- removed link Gripper_2
- added link pointer_base, mass 0.1; collision cylinder length=0.05 radius=0.025; visual cylinder length=0.05 radius=0.025
- added link pointer_tip, mass 0.03; collision cylinder length=0.05 radius=0.012; collision sphere radius=0.008
Joints:
- removed joint Finger_1
- removed joint Finger_2
- added joint pointer_base_joint: type fixed, parent Link_6, child pointer_base, origin xyz=0 -0.05 0.05 rpy=0 0 0
- added joint pointer_extend_joint: type prismatic, parent pointer_base, child pointer_tip, origin xyz=0 0 0.05 rpy=0 0 0, axis 0 0 1, limit lower=0 upper=0.05 effort=50 velocity=5
